File: KeyPad.kicad_pcb (KiCad board)
At the start: 2 copper layers, 41.9 x 41.9 mm, 16 parts, among them P1 CONN_01X03, SW1 SW_Push_Dual, SW2 SW_Push_Dual, SW3 SW_Push_Dual, SW4 SW_Push_Dual

Commit message: conector cambiado
Parts:
- P1: footprint Connectors_JST:JST_PH_S3B-PH-K_03x2.00mm_Angled -> lib_fp:JST_PH_S3B-PH-K_03x2.00mm_Angled
- R1, R2, R3, R4: footprint Resistors_SMD:R_0805 -> lib_fp:R_0805
- SW1, SW2, SW3, SW4: footprint Buttons_Switches_THT:SW_PUSH-12mm -> lib_fp:SW_PUSH-12mm
- moved P1 0.16 mm to (152.6, 119.4)
Connections:
- P1 pad 1: GND -> Net-(P1-Pad1)
- P1 pad 3: Net-(P1-Pad3) -> GND
- R1 pad 2: Net-(P1-Pad3) -> Net-(P1-Pad1)
- R2 pad 1: Net-(P1-Pad3) -> Net-(P1-Pad1)
- SW1 pad 1: Net-(SW1-Pad1) -> Net-(P1-Pad1)
Routing:
- net Net-(P1-Pad1): track 0.00 -> 50.3 mm
- net Net-(P1-Pad3): track 38.4 -> 0.00 mm
- net Net-(SW1-Pad1): track 17.7 -> 0.00 mm
- net VCC: track 26.6 -> 27.7 mm
